File: pcb/vindriktrning-esp32-s3/vindriktrning-esp32-s3.kicad_pcb (KiCad board)
At the start: 4 copper layers, 39 x 74.5 mm, 43 parts, among them IC1 SCD30, J1 P2.5, J2 Conn_01x01_Pin, Q1 AO3400A_C347475, Q2 BSD840NH6327XTSA1, Q3 BSS138, SW1 RESET Swtich, SW2 BOOT Switch, U1 SMD0805-20, U2 D1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

Commit message: wip
Parts:
- added J10: Conn_01x01_Pin, TestPoint:TestPoint_Pad_D1.0mm, F.Cu at (102.9, 114.0)
- added J11: Conn_01x01_Pin, TestPoint:TestPoint_Pad_D1.0mm, F.Cu at (102.5, 108.6)
- added J3: Conn_01x01_Pin, TestPoint:TestPoint_Pad_D1.0mm, F.Cu at (97.7, 103.3)
- added J4: Conn_01x01_Pin, TestPoint:TestPoint_Pad_D1.0mm, F.Cu at (93.7, 103.3)
- added J5: Conn_01x01_Pin, TestPoint:TestPoint_Pad_D1.0mm, F.Cu at (94.8, 119.1)
- added J6: Conn_01x01_Pin, TestPoint:TestPoint_Pad_D1.0mm, F.Cu at (99.1, 121.3)
- added J7: Conn_01x01_Pin, TestPoint:TestPoint_Pad_D1.0mm, F.Cu at (101.4, 120.1)
- added J8: Conn_01x01_Pin, TestPoint:TestPoint_Pad_D1.0mm, F.Cu at (102.7, 118.5)
- added J9: Conn_01x01_Pin, TestPoint:TestPoint_Pad_D1.0mm, F.Cu at (102.8, 116.2)
- moved J2 23.6 mm to (95.7, 103.3)
Connections:
- J2 pad 1: unconnected-(J2-Pin_1-Pad1) -> TXD0
- U6 pad 15: FAN -> IO6
- U6 pad 26: IO20 -> FAN
Routing:
- net LIGHT: track 16.0 -> 62.6 mm, vias 1 -> 2
- net FAN: track 0.00 -> 16.3 mm
- net IO3: track 0.00 -> 5.91 mm, vias 0 -> 2
- net IO0: track 0.00 -> 4.65 mm
- net IO1: track 0.00 -> 4.20 mm
- net RXD0: track 0.00 -> 3.39 mm
- net IO6: track 0.00 -> 3.39 mm
- net IO7: track 0.00 -> 2.47 mm
- net TXD0: track 0.00 -> 2.43 mm
- net +5V: track 154.9 -> 156.9 mm, vias 4 -> 5
- net IO2: track 0.00 -> 1.88 mm
- net IO8: track 0.00 -> 1.79 mm
- net GND: vias 8 -> 13
Other:
- board text added: "0V"
- board text added: "3V"
- board text added: "5V"
- board text added: "BOOT"
- board text added: "RESET"
- board text added: "RX"
- board text added: "SCL"
- board text added: "SDA"
- board text added: "TX"
