File: pcb/vindriktrning-esp32-s3/vindriktrning-esp32-s3.kicad_sch (KiCad schematic)
At the start: 43 parts, among them IC1 SCD30, J1 P2.5, J2 Conn_01x01_Pin, Q1 AO3400A_C347475, Q2 BSD840NH6327XTSA1, Q3 BSS138, SW1 RESET Swtich, SW2 BOOT Switch, U1 SMD0805-20, U2 D1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

Commit message: wip
Parts:
- added J10, J11, J3, J4, J5, J6, J7, J8, J9: Conn_01x01_Pin, TestPoint:TestPoint_Pad_D1.0mm, symbol Connector:Conn_01x01_Pin
- C1: LCSC (none) -> C335982
- C2, C3: LCSC (none) -> C15850
- C4: LCSC (none) -> C1710
- C5: LCSC (none) -> C28323
- FAN1: LCSC (none) -> C393945
- J1: LCSC (none) -> C145997
- LED1, LED2, LED3, LED4: LCSC (none) -> C5349954
- Q1: LCSC (none) -> C347475
- Q2: LCSC (none) -> C151516
- Q3: LCSC (none) -> C5224263
- R1, R11, R12, R13, R5: LCSC (none) -> C23186
- R10, R14, R2, R7, R8, R9: LCSC (none) -> C25804
- R15: LCSC (none) -> C21190
- R16, R3, R4, R6: LCSC (none) -> C25803
- SW1, SW2: LCSC (none) -> C720477
- U1: LCSC (none) -> C250858
- U2: LCSC (none) -> C917121
- U3: LCSC (none) -> C2891705
- U4: LCSC (none) -> C841192
- U6: LCSC (none) -> C5736265
- USB1: LCSC (none) -> C7450621
Connections:
- net IO20 is gone; now on net FAN: U6.26 (IO20)
- net FAN: no longer U6.15 (IO6)
- net GND: now also J4.1 (Pin_1)
- net IO0: now also J7.1 (Pin_1)
- net IO1: now also J8.1 (Pin_1)
- net IO2: now also J5.1 (Pin_1)
- net IO3: now also J6.1 (Pin_1)
- net IO7: now also J10.1 (Pin_1)
- net IO8: now also J11.1 (Pin_1)
- net RXD0: now also J3.1 (Pin_1)
- net TXD0: now also J2.1 (Pin_1)
- new net IO6: J9.1 (Pin_1), U6.15 (IO6)
